Commit message: Update RoboSimian model to new URDF specification

File: data/robosimian/rs_new.urdf (robot description, URDF)
Before this commit: robot robosim, 72 links, 71 joints
Links:
- removed link dd_wheel_left
- removed link dd_wheel_right
- removed link limb1_finger0_link0
- removed link limb1_finger0_link_actuator
- removed link limb1_finger1_link0
- removed link limb1_finger1_link_actuator
- removed link limb1_finger2_link0
- removed link limb1_finger2_link_actuator
- removed link limb2_finger0_link0
- removed link limb2_finger0_link_actuator
- removed link limb2_finger1_link0
- removed link limb2_finger1_link_actuator
- removed link limb2_finger2_link0
- removed link limb2_finger2_link_actuator
- removed link limb3_finger0_link0
- removed link limb3_finger0_link_actuator
- removed link limb3_finger1_link0
- removed link limb3_finger1_link_actuator
- removed link limb3_finger2_link0
- removed link limb3_finger2_link_actuator
- removed link limb4_finger0_link0
- removed link limb4_finger0_link_actuator
- removed link limb4_finger1_link0
- removed link limb4_finger1_link_actuator
- removed link limb4_finger2_link0
- removed link limb4_finger2_link_actuator
- added link sled, mass 2.769; collision cylinder length=0.145 radius=0.05; visual mesh filename=./stl/robosim_sled_new.stl scale=1 1 1
- link limb1_ft_link: mass 3.975000 -> 0.1492
- link limb1_ftadapter_link: mass 3.975000 -> 0.2242
- link limb1_link7: mass 1.760000 -> 3.1775
- link limb1_link8: mass 1.760000 -> 1.2
- link limb2_ft_link: mass 3.975000 -> 0.1492
- link limb2_ftadapter_link: mass 3.975000 -> 0.2242
- link limb2_link7: mass 1.760000 -> 3.1775
- link limb2_link8: mass 1.760000 -> 1.2
- link limb3_ft_link: mass 3.975000 -> 0.1492
- link limb3_ftadapter_link: mass 3.975000 -> 0.2242
- link limb3_link7: mass 1.760000 -> 3.1775
- link limb3_link8: mass 1.760000 -> 1.2
- link limb4_ft_link: mass 3.975000 -> 0.1492
- link limb4_ftadapter_link: mass 3.975000 -> 0.2242
- link limb4_link7: mass 1.760000 -> 3.1775
- link limb4_link8: mass 1.760000 -> 1.2
Joints:
- removed joint dd_left
- removed joint dd_right
- removed joint limb1_finger0_actuator
- removed joint limb1_finger0_joint0
- removed joint limb1_finger1_actuator
- removed joint limb1_finger1_joint0
- removed joint limb1_finger2_actuator
- removed joint limb1_finger2_joint0
- removed joint limb2_finger0_actuator
- removed joint limb2_finger0_joint0
- removed joint limb2_finger1_actuator
- removed joint limb2_finger1_joint0
- removed joint limb2_finger2_actuator
- removed joint limb2_finger2_joint0
- removed joint limb3_finger0_actuator
- removed joint limb3_finger0_joint0
- removed joint limb3_finger1_actuator
- removed joint limb3_finger1_joint0
- removed joint limb3_finger2_actuator
- removed joint limb3_finger2_joint0
- removed joint limb4_finger0_actuator
- removed joint limb4_finger0_joint0
- removed joint limb4_finger1_actuator
- removed joint limb4_finger1_joint0
- removed joint limb4_finger2_actuator
- removed joint limb4_finger2_joint0
- added joint sled_joint: type fixed, parent torso, child sled, origin xyz=0.0 0.0 0.21 rpy=1.570796 0.00 0.00
- joint base_to_torso: origin xyz=0 0.0 0.0 rpy=0.0 0.0 0.0 -> xyz=0 0.0 0.0 rpy=3.14159 0.0 0.0
