Commit message: Update to latest URDF description (inertia provided in centroidal frames)

File: data/robosimian/rs.urdf (robot description, URDF)
Before this commit: robot robosim, 72 links, 71 joints
Links:
- removed link dd_wheel_left
- removed link dd_wheel_right
- removed link limb1_finger0_link0
- removed link limb1_finger0_link_actuator
- removed link limb1_finger1_link0
- removed link limb1_finger1_link_actuator
- removed link limb1_finger2_link0
- removed link limb1_finger2_link_actuator
- removed link limb2_finger0_link0
- removed link limb2_finger0_link_actuator
- removed link limb2_finger1_link0
- removed link limb2_finger1_link_actuator
- removed link limb2_finger2_link0
- removed link limb2_finger2_link_actuator
- removed link limb3_finger0_link0
- removed link limb3_finger0_link_actuator
- removed link limb3_finger1_link0
- removed link limb3_finger1_link_actuator
- removed link limb3_finger2_link0
- removed link limb3_finger2_link_actuator
- removed link limb4_finger0_link0
- removed link limb4_finger0_link_actuator
- removed link limb4_finger1_link0
- removed link limb4_finger1_link_actuator
- removed link limb4_finger2_link0
- removed link limb4_finger2_link_actuator
- added link sled, mass 2.768775; collision mesh filename=./stl/robosim_sled.stl scale=1 1 1; visual mesh filename=./stl/robosim_sled.stl scale=1 1 1
- link limb1_ft_link: mass 3.975000 -> 0.195418
- link limb1_ftadapter_link: mass 3.975000 -> 0.253735
- link limb1_link1: mass 0.429000 -> 0.428770
- link limb1_link2: mass 3.975000 -> 4.078540
- link limb1_link3: mass 0.429000 -> 0.428770
- link limb1_link4: mass 3.975000 -> 4.078540
- link limb1_link5: mass 0.429000 -> 0.428770
- link limb1_link6: mass 3.975000 -> 4.078540
- link limb1_link7: mass 1.760000 -> 3.1775
- link limb1_link8: mass 1.760000 -> 1.499326
- link limb2_ft_link: mass 3.975000 -> 0.195418
- link limb2_ftadapter_link: mass 3.975000 -> 0.253735
- link limb2_link1: mass 0.429000 -> 0.428770
- link limb2_link2: mass 3.975000 -> 4.078540
- link limb2_link3: mass 0.429000 -> 0.428770
- link limb2_link4: mass 3.975000 -> 4.078540
- link limb2_link5: mass 0.429000 -> 0.428770
- link limb2_link6: mass 3.975000 -> 4.078540
- link limb2_link7: mass 1.760000 -> 3.1775
- link limb2_link8: mass 1.760000 -> 1.499326
- link limb3_ft_link: mass 3.975000 -> 0.195418
- link limb3_ftadapter_link: mass 3.975000 -> 0.253735
- link limb3_link1: mass 0.429000 -> 0.428770
- link limb3_link2: mass 3.975000 -> 4.078540
- link limb3_link3: mass 0.429000 -> 0.428770
- link limb3_link4: mass 3.975000 -> 4.078540
- link limb3_link5: mass 0.429000 -> 0.428770
- link limb3_link6: mass 3.975000 -> 4.078540
- link limb3_link7: mass 1.760000 -> 3.1775
- link limb3_link8: mass 1.760000 -> 1.499326
- link limb4_ft_link: mass 3.975000 -> 0.195418
- link limb4_ftadapter_link: mass 3.975000 -> 0.253735
- link limb4_link1: mass 0.429000 -> 0.428770
- link limb4_link2: mass 3.975000 -> 4.078540
- link limb4_link3: mass 0.429000 -> 0.428770
- link limb4_link4: mass 3.975000 -> 4.078540
- link limb4_link5: mass 0.429000 -> 0.428770
- link limb4_link6: mass 3.975000 -> 4.078540
- link limb4_link7: mass 1.760000 -> 3.1775
- link limb4_link8: mass 1.760000 -> 1.499326
- link torso: mass 40.000000 -> 46.658335
Joints:
- removed joint dd_left
- removed joint dd_right
- removed joint limb1_finger0_actuator
- removed joint limb1_finger0_joint0
- removed joint limb1_finger1_actuator
- removed joint limb1_finger1_joint0
- removed joint limb1_finger2_actuator
- removed joint limb1_finger2_joint0
- removed joint limb2_finger0_actuator
- removed joint limb2_finger0_joint0
- removed joint limb2_finger1_actuator
- removed joint limb2_finger1_joint0
- removed joint limb2_finger2_actuator
- removed joint limb2_finger2_joint0
- removed joint limb3_finger0_actuator
- removed joint limb3_finger0_joint0
- removed joint limb3_finger1_actuator
- removed joint limb3_finger1_joint0
- removed joint limb3_finger2_actuator
- removed joint limb3_finger2_joint0
- removed joint limb4_finger0_actuator
- removed joint limb4_finger0_joint0
- removed joint limb4_finger1_actuator
- removed joint limb4_finger1_joint0
- removed joint limb4_finger2_actuator
- removed joint limb4_finger2_joint0
- added joint sled_joint: type fixed, parent torso, child sled, origin xyz=0.0 0.0 0.21 rpy=1.570796 0.00 0.00

Commit message: Fixes to collision geometry for RoboSimian.
- use new convex mesh for sled collision geometry
- ensure all collision family settings are done *before* enabliung collision for a body (order important for Chrono::Parallel)

File: data/robosimian/rs.urdf (robot description, URDF)
Before this commit: robot robosim, 47 links, 46 joints
Links:
- link sled: geometry collision mesh filename=./stl/robosim_sled_coll.stl scale=1 1 1; visual mesh filename=./stl/robosim_sled.stl scale=1 1 1
